File: alimentation.kicad_sch (KiCad schematic)
At the start: 8 parts, among them J2 12.0, M1 Convertisseur 3V3, M2 Convertisseur 5V, Q1 FQP27P06

Commit message: PCB me parrait OK
Parts:
- removed M1: Convertisseur 3V3, library:MP1584EN, symbol New_Library:DC_DC_Converter
- D2: footprint Diode_THT:D_DO-15_P12.70mm_Horizontal -> Diode_SMD:D_SMB_Handsoldering
- J2: footprint Connector_BarrelJack:BarrelJack_CUI_PJ-036AH-SMT_Horizontal -> Connector_BarrelJack:BarrelJack_GCT_DCJ200-10-A_Horizontal; symbol Connector:Jack-DC -> Connector:Barrel_Jack_Switch
Connections:
- net +12V: now also Q1.3 (S); no longer Q1.2 (D)
- net GND: now also J2.2; no longer J2.1
- net at F1.2: now also J2.1; no longer J2.2
- net at Q1.1 (G), R2.2: now also D1.1 (K); no longer D1.2 (A)
- new net: D1.2 (A), F1.1, Q1.2 (D)
Other:
- note added: "Alimentation 12V"
- note removed: "Alimentation 12V A revevoir + stabilité"
- moved on the sheet: D1, D2, F1, M2, Q1, R2
