File: ihm.kicad_sch (KiCad schematic)
At the start: 13 parts, among them Q11 2N2219, SW1 SW_Push

Commit message: PCB me parrait OK
Parts:
- removed D5, D6: LED, LED_THT:LED_D3.0mm, symbol Device:LED
- removed R41, R42: R 500, Resistor_THT:R_Axial_DIN0207_L6.3mm_D2.5mm_P7.62mm_Horizontal, symbol Device:R
- BZ1: footprint (none) -> library:buzzer
