File: medbox.kicad_pcb (KiCad board)
At the start: 2 copper layers, 34 parts, among them J1 Connecteur moteur pas a pas, J2 12.0, M1 Convertisseur 3V3, M2 Convertisseur 5V, M3 Connecteur module RTC, Q1 FQP27P06, Q11 2N2219, SW1 SW_Push, U4 ESP32-DevKitC

Commit message: update pcb
Parts:
- removed J1: Connecteur moteur pas a pas, Connector_JST:JST_PH_B6B-PH-K_1x06_P2.00mm_Vertical
- added J3: Connecteur moteur pas a pas, Connector_JST:JST_PH_B6B-PH-K_1x06_P2.00mm_Vertical, F.Cu at (63.0, 171.0)
Connections:
- U4 pad 12: MOT_MS3 -> unconnected-(U4-MTMS/GPIO14/ADC2_CH6-Pad12)
- U4 pad 23: LED_MEDIC -> unconnected-(U4-MTDO/GPIO15/ADC2_CH3-Pad23)
- U4 pad 26: GAT_LED_POWER -> unconnected-(U4-ADC2_CH0/GPIO4-Pad26)
- U4 pad 27: unconnected-(U4-GPIO16-Pad27) -> MOT_MS3
- U4 pad 28: unconnected-(U4-GPIO17-Pad28) -> LED_MEDIC

Commit message: PCB me parrait OK
Parts:
- removed C4: C, Capacitor_THT:C_Disc_D5.0mm_W2.5mm_P2.50mm
- removed D5, D6: LED, LED_THT:LED_D3.0mm
- removed M1: Convertisseur 3V3, library:MP1584EN
- removed R41, R42: R 500, Resistor_THT:R_Axial_DIN0207_L6.3mm_D2.5mm_P7.62mm_Horizontal
- added BZ1: Buzzer, library:buzzer, F.Cu at (97.5, 136.0)
- added REF**: MountingHole_2.2mm_M2, MountingHole:MountingHole_2.2mm_M2, F.Cu at (174.5, 67.5)
- added REF**: MountingHole_2.2mm_M2, MountingHole:MountingHole_2.2mm_M2, F.Cu at (78.0, 73.5)
- added REF**: MountingHole_2.2mm_M2, MountingHole:MountingHole_2.2mm_M2, F.Cu at (145.5, 88.0)
- added REF**: MountingHole_2.2mm_M2, MountingHole:MountingHole_2.2mm_M2, F.Cu at (64.5, 147.0)
- C1: footprint Capacitor_THT:CP_Radial_D6.3mm_P2.50mm -> Capacitor_THT:CP_Radial_D10.0mm_P5.00mm
- C2, C3: footprint Capacitor_THT:C_Disc_D5.0mm_W2.5mm_P2.50mm -> Capacitor_THT:C_Disc_D6.0mm_W2.5mm_P5.00mm
- D2: footprint Diode_THT:D_DO-15_P12.70mm_Horizontal -> Diode_SMD:D_SMB_Handsoldering
- J2: footprint Connector_BarrelJack:BarrelJack_CUI_PJ-036AH-SMT_Horizontal -> Connector_BarrelJack:BarrelJack_GCT_DCJ200-10-A_Horizontal
- moved C1 252.0 mm to (143.0, 67.3), turned to -90 degrees
- moved C3 237.9 mm to (135.8, 83.2), turned to -90 degrees
- moved C2 236.8 mm to (135.0, 70.5), turned to 90 degrees
- moved R1 181.1 mm to (93.3, 164.0), turned to 180 degrees
- moved D7 166.4 mm to (91.6, 174.6), turned to 150 degrees
- moved D3 165.5 mm to (90.0, 146.6), turned to 90 degrees
- moved M3 161.1 mm to (72.2, 136.5), turned to 90 degrees
- moved Q11 159.0 mm to (87.0, 155.0)
- moved J3 147.8 mm to (187.0, 90.5), turned to 180 degrees
- moved R40 143.7 mm to (86.0, 145.3), turned to 90 degrees
- moved F1 131.1 mm to (122.5, 48.0)
- moved J2 130.4 mm to (112.5, 53.0), turned to 180 degrees
- moved D1 130.3 mm to (128.2, 54.5), turned to 0 degrees
- moved D4 122.4 mm to (85.0, 171.8), turned to 140 degrees
- moved Q1 121.8 mm to (129.4, 49.5), turned to 0 degrees
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Connections:
- C1 pad 1: GND -> +12V
- C1 pad 2: +12V -> GND
- F1 pad 1: Net-(D1-K) -> Net-(D1-A)
- J2 pad 1: GND -> Net-(F1-Pad2)
- J2 pad 2: Net-(F1-Pad2) -> GND
- J2 pad 3: (no net) -> unconnected-(J2-Pad3)
- J3 pad 1: Net-(A1-1A) -> Net-(A1-2B)
- J3 pad 3: Net-(A1-1B) -> Net-(A1-2A)
- J3 pad 4: Net-(A1-2A) -> Net-(A1-1B)
- J3 pad 6: Net-(A1-2B) -> Net-(A1-1A)
- M3 pad 2: +3.3V -> +3V3
- Q1 pad 1: Net-(D1-A) -> Net-(D1-K)
- Q1 pad 2: +12V -> Net-(D1-A)
- Q1 pad 3: Net-(D1-K) -> +12V
- R13 pad 1: MOT_MS1 -> GND
- R13 pad 2: GND -> MOT_MS1
- R2 pad 2: Net-(D1-A) -> Net-(D1-K)
- R3 pad 1: +3V3 -> MOT_ENABLED
- R3 pad 2: MOT_ENABLED -> +3V3
- R9 pad 1: +3V3 -> Net-(A1-~{SLEEP})
- R9 pad 2: Net-(A1-~{SLEEP}) -> +3V3
- U4 pad 1: unconnected-(U4-3V3-Pad1) -> GND
- U4 pad 10: LED_WIFI -> unconnected-(U4-DAC_1/ADC2_CH8/GPIO25-Pad10)
- U4 pad 11: MOT_ENABLED -> unconnected-(U4-DAC_2/ADC2_CH9/GPIO26-Pad11)
- U4 pad 12: unconnected-(U4-MTMS/GPIO14/ADC2_CH6-Pad12) -> MOT_ENABLED
- U4 pad 13: MOT_MS2 -> MOT_MS3
- U4 pad 14: GND -> MOT_MS2
- U4 pad 16: unconnected-(U4-SD_DATA2/GPIO9-Pad16) -> MOT_MS1
- U4 pad 2: unconnected-(U4-CHIP_PU-Pad2) -> +3V3
- U4 pad 24: LED_STATUS -> LED_POWER
- U4 pad 26: unconnected-(U4-ADC2_CH0/GPIO4-Pad26) -> TRIGGER_BTN
- U4 pad 27: MOT_MS3 -> unconnected-(U4-GPIO16-Pad27)
- U4 pad 3: TRIGGER_BTN -> unconnected-(U4-EN-Pad3)
- U4 pad 6: ANY_FAIL -> unconnected-(U4-VDET_1/GPIO34/ADC1_CH6-Pad6)
- U4 pad 7: MOT_DIR -> unconnected-(U4-VDET_2/GPIO35/ADC1_CH7-Pad7)
- U4 pad 8: MOT_STEP -> MOT_DIR
- U4 pad 9: LED_POWER -> MOT_STEP
Routing:
- net GND: track 0.00 -> 380.4 mm, vias 0 -> 1
- net +3V3: track 0.00 -> 197.0 mm, vias 0 -> 3
- net TRIGGER_BTN: track 0.00 -> 89.9 mm, vias 0 -> 2
- net PILOTAGE_BUZ: track 0.00 -> 77.9 mm
- net Net-(A1-2B): track 0.00 -> 68.4 mm
- net Net-(A1-2A): track 0.00 -> 63.6 mm
- net Net-(D7-A): track 0.00 -> 59.8 mm
- net +5V: track 0.00 -> 59.5 mm
- net Net-(A1-1B): track 0.00 -> 58.5 mm
- net Net-(A1-1A): track 0.00 -> 57.5 mm, vias 0 -> 1
- net LED_POWER: track 0.00 -> 54.6 mm
- net +12V: track 0.00 -> 49.8 mm
- net MOT_DIR: track 91.8 -> 42.2 mm
- net MOT_STEP: track 89.8 -> 42.2 mm
- net MOT_ENABLED: track 103.4 -> 61.9 mm, vias 2 -> 1
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- added copper zone on B.Cu, net GND
Other:
- board outline added: 141.2 x 137.9 mm
