File: medbox.kicad_sch (KiCad schematic)
At the start: 3 parts, among them M3 Connecteur module RTC, U4 ESP32-DevKitC

Commit message: update pcb
Connections:
- net LED_MEDIC: now also U4.28 (GPIO17); no longer U4.23 (MTDO/GPIO15/ADC2_CH3)
- net MOT_MS3: now also U4.27 (GPIO16); no longer U4.12 (MTMS/GPIO14/ADC2_CH6)
- net GAT_LED_POWER: no longer names the net of U4.26 (ADC2_CH0/GPIO4)
Changed lines of the file:
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@@
+	(wire
+		(pts
+			(xy 226.06 107.95) (xy 231.14 107.95)
+		)
+		(stroke
+			(width 0)
+			(type default)
+		)
+	)
 	(wire
 		(pts
@@
 	(wire
 		(pts
-			(xy 153.67 69.85) (xy 160.02 69.85)
-		)
-		(stroke
-			(width 0)
-			(type default)
-		)
-	)
-	(wire
-		(pts
 			(xy 226.06 85.09) (xy 231.14 85.09)
 		)
@@
 	(wire
 		(pts
-			(xy 226.06 62.23) (xy 229.87 62.23)
+			(xy 226.06 110.49) (xy 231.14 110.49)
 		)
 		(stroke
@@
 		)
 	)
-	(wire
-		(pts
-			(xy 153.67 67.31) (xy 160.02 67.31)
-		)
-		(stroke
-			(width 0)
-			(type default)
-		)
-	)
 	(global_label "ANY_FAIL"
 		(shape input)
@@
 	(global_label "MOT_MS3"
 		(shape input)
-		(at 153.67 67.31 180)
+		(at 231.14 107.95 0)
+		(fields_autoplaced yes)
+		(effects
+			(font
+				(size 1.27 1.27)
+			)
+			(justify left)
+		)
+		(property "Intersheetrefs" "${INTERSHEET_REFS}"
+			(at 242.7127 107.95 0)
+			(effects
+				(font
+					(size 1.27 1.27)
+				)
+				(justify left)
+				(hide yes)
+			)
+		)
+	)
+	(global_label "LED_WIFI"
+		(shape input)
+		(at 231.14 82.55 0)
+		(fields_autoplaced yes)
+		(effects
+			(font
+				(size 1.27 1.27)
+			)
+			(justify left)
+		)
+		(property "Intersheetrefs" "${INTERSHEET_REFS}"
+			(at 242.2895 82.55 0)
+			(effects
+				(font
+					(size 1.27 1.27)
+				)
+				(justify left)
+				(hide yes)
+			)
+		)
+	)
+	(global_label "LED_MEDIC"
+		(shape input)
+		(at 231.14 110.49 0)
+		(fields_autoplaced yes)
+		(effects
+			(font
+				(size 1.27 1.27)
+			)
+			(justify left)
+		)
+		(property "Intersheetrefs" "${INTERSHEET_REFS}"
+			(at 244.2851 110.49 0)
+			(effects
+				(font
+					(size 1.27 1.27)
+				)
+				(justify left)
+				(hide yes)
+			)
+		)
+	)
+	(global_label "I2C_SDA"
+		(shape input)
+		(at 231.14 72.39 0)
+		(fields_autoplaced yes)
+		(effects
+			(font
+				(size 1.27 1.27)
+			)
+			(justify left)
+		)
+		(property "Intersheetrefs" "${INTERSHEET_REFS}"
+			(at 241.7452 72.39 0)
+			(effects
+				(font
+					(size 1.27 1.27)
+				)
+				(justify left)
+				(hide yes)
+			)
+		)
+	)
+	(global_label "PILOTAGE_BUZ"
+		(shape input)
+		(at 229.87 64.77 0)
+		(fields_autoplaced yes)
+		(effects
+			(font
+				(size 1.27 1.27)
+			)
+			(justify left)
+		)
+		(property "Intersheetrefs" "${INTERSHEET_REFS}"
+			(at 246.3414 64.77 0)
+			(effects
+				(font
+					(size 1.27 1.27)
+				)
+				(justify left)
+				(hide yes)
+			)
+		)
+	)
+	(global_label "LED_POWER"
+		(shape input)
+		(at 231.14 80.01 0)
+		(fields_autoplaced yes)
+		(effects
+			(font
+				(size 1.27 1.27)
+			)
+			(justify left)
+		)
+		(property "Intersheetrefs" "${INTERSHEET_REFS}"
+			(at 245.0108 80.01 0)
+			(effects
+				(font
+					(size 1.27 1.27)
+				)
+				(justify left)
+				(hide yes)
+			)
+		)
+	)
+	(global_label "MOT_DIR"
+		(shape input)
+		(at 153.67 54.61 180)
 		(fields_autoplaced yes)
 		(effects
@@
 		)
 		(property "Intersheetrefs" "${INTERSHEET_REFS}"
-			(at 142.0973 67.31 0)
+			(at 142.8229 54.61 0)
 			(effects
 				(font
@@
 		)
 	)
-	(global_label "LED_WIFI"
-		(shape input)
-		(at 231.14 82.55 0)
-		(fields_autoplaced yes)
-		(effects
-			(font
-				(size 1.27 1.27)
-			)
-			(justify left)
-		)
-		(property "Intersheetrefs" "${INTERSHEET_REFS}"
-			(at 242.2895 82.55 0)
-			(effects
-				(font
-					(size 1.27 1.27)
-				)
-				(justify left)
-				(hide yes)
-			)
-		)
-	)
-	(global_label "LED_MEDIC"
-		(shape input)
-		(at 153.67 69.85 180)
+	(global_label "MOT_ENABLED"
+		(shape input)
+		(at 231.14 85.09 0)
+		(fields_autoplaced yes)
+		(effects
+			(font
+				(size 1.27 1.27)
+			)
+			(justify left)
+		)
+		(property "Intersheetrefs" "${INTERSHEET_REFS}"
+			(at 247.1275 85.09 0)
+			(effects
+				(font
+					(size 1.27 1.27)
+				)
+				(justify left)
+				(hide yes)
+			)
+		)
+	)
+	(global_label "MOT_STEP"
+		(shape input)
+		(at 153.67 57.15 180)
 		(fields_autoplaced yes)
 		(effects
@@
 		)
 		(property "Intersheetrefs" "${INTERSHEET_REFS}"
-			(at 140.5249 69.85 0)
+			(at 141.3716 57.15 0)
 			(effects
 				(font
@@
 				(hide yes)
 			)
-		)
-	)
-	(global_label "I2C_SDA"
-		(shape input)
-		(at 231.14 72.39 0)
-		(fields_autoplaced yes)
-		(effects
-			(font
-				(size 1.27 1.27)
-			)
-			(justify left)
-		)
-		(property "Intersheetrefs" "${INTERSHEET_REFS}"
-			(at 241.7452 72.39 0)
-			(effects
-				(font
-					(size 1.27 1.27)
-				)
-				(justify left)
-				(hide yes)
-			)
-		)
-	)
-	(global_label "PILOTAGE_BUZ"
-		(shape input)
-		(at 229.87 64.77 0)
-		(fields_autoplaced yes)
-		(effects
-			(font
-				(size 1.27 1.27)
-			)
-			(justify left)
-		)
-		(property "Intersheetrefs" "${INTERSHEET_REFS}"
-			(at 246.3414 64.77 0)
-			(effects
-				(font
-					(size 1.27 1.27)
-				)
-				(justify left)
-				(hide yes)
-			)
-		)
-	)
-	(global_label "LED_POWER"
-		(shape input)
-		(at 231.14 80.01 0)
-		(fields_autoplaced yes)
-		(effects
-			(font
-				(size 1.27 1.27)
-			)
-			(justify left)
-		)
-		(property "Intersheetrefs" "${INTERSHEET_REFS}"
-			(at 245.0108 80.01 0)
-			(effects
-				(font
-					(size 1.27 1.27)
-				)
-				(justify left)
-				(hide yes)
-			)
-		)
-	)
-	(global_label "MOT_DIR"
-		(shape input)
-		(at 153.67 54.61 180)
-		(fields_autoplaced yes)
-		(effects
-			(font
-				(size 1.27 1.27)
-			)
-			(justify right)
-		)
-		(property "Intersheetrefs" "${INTERSHEET_REFS}"
-			(at 142.8229 54.61 0)
-			(effects
-				(font
-					(size 1.27 1.27)
-				)
-				(justify right)
-				(hide yes)
-			)
-		)
-	)
-	(global_label "MOT_ENABLED"
-		(shape input)
-		(at 231.14 85.09 0)
-		(fields_autoplaced yes)
-		(effects
-			(font
-				(size 1.27 1.27)
-			)
-			(justify left)
-		)
-		(property "Intersheetrefs" "${INTERSHEET_REFS}"
-			(at 247.1275 85.09 0)
-			(effects
-				(font
-					(size 1.27 1.27)
-				)
-				(justify left)
-				(hide yes)
-			)
-		)
-	)
-	(global_label "MOT_STEP"
-		(shape input)
-		(at 153.67 57.15 180)
-		(fields_autoplaced yes)
-		(effects
-			(font
-				(size 1.27 1.27)
-			)
-			(justify right)
-		)
-		(property "Intersheetrefs" "${INTERSHEET_REFS}"
-			(at 141.3716 57.15 0)
-			(effects
-				(font
-					(size 1.27 1.27)
-				)
-				(justify right)
-				(hide yes)
-			)
-		)
-	)
-	(global_label "GAT_LED_POWER"
-		(shape input)
-		(at 229.87 62.23 0)
-		(fields_autoplaced yes)
-		(effects
-			(font
-				(size 1.27 1.27)
-			)
-			(justify left)
-		)
-		(property "Intersheetrefs" "${INTERSHEET_REFS}"
-			(at 248.0346 62.23 0)
-			(effects
-				(font
-					(size 1.27 1.27)
-				)
-				(justify left)
-				(hide yes)
-			)

Commit message: PCB me parrait OK
Parts:
- removed C4: C, Capacitor_THT:C_Disc_D5.0mm_W2.5mm_P2.50mm, symbol Device:C
Connections:
- net +3.3V is gone; now on net +3V3: M3.2 (VCC)
- net LED_STATUS is gone; now on net LED_POWER: U4.24 (ADC2_CH2/GPIO2)
- net +5V: now also U4.0 (5V); no longer U4.19 (5V)
- net GND: now also U4.1 (GND); no longer U4.14 (GND), U4.32 (GND), U4.38 (GND)
- net LED_POWER: no longer U4.9 (DAC_1/ADC2_CH8/GPIO25)
- net MOT_DIR: now also U4.8 (32K_XP/GPIO32/ADC1_CH4); no longer U4.7 (32K_XP/GPIO32/ADC1_CH4)
- net MOT_ENABLED: now also U4.12 (ADC2_CH7/GPIO27); no longer U4.11 (ADC2_CH7/GPIO27)
- net MOT_MS1: now also U4.16 (MTCK/GPIO13/ADC2_CH4); no longer U4.15 (MTCK/GPIO13/ADC2_CH4)
- net MOT_MS2: now also U4.14 (MTDI/GPIO12/ADC2_CH5); no longer U4.13 (MTDI/GPIO12/ADC2_CH5)
- net MOT_MS3: now also U4.13 (MTMS/GPIO14/ADC2_CH6); no longer U4.27 (GPIO16)
- net MOT_STEP: now also U4.9 (32K_XN/GPIO33/ADC1_CH5); no longer U4.8 (32K_XN/GPIO33/ADC1_CH5)
- net TRIGGER_BTN: now also U4.26 (ADC2_CH0/GPIO4); no longer U4.3 (SENSOR_VP/GPIO36/ADC1_CH0)
- net +3V3: now reaches U4.2 (3V3)
- net ANY_FAIL: no longer names the net of U4.6 (VDET_1/GPIO34/ADC1_CH6)
- net LED_WIFI: no longer names the net of U4.10 (DAC_1/ADC2_CH8/GPIO25)
- new net: U4.32 (GND), U4.38 (GND)
