File: pilotage_moteur.kicad_sch (KiCad schematic)
At the start: 11 parts, among them J1 Connecteur moteur pas a pas

Commit message: update pcb
Parts:
- removed J1: Connecteur moteur pas a pas, Connector_JST:JST_PH_B6B-PH-K_1x06_P2.00mm_Vertical, symbol Connector:Conn_01x04_Socket
- added J3: Connecteur moteur pas a pas, Connector_JST:JST_PH_B6B-PH-K_1x06_P2.00mm_Vertical, symbol Connector:Conn_01x06_Socket
Connections:
- net at A1.3 (1B): now also J3.3 (Pin_3)
- net at A1.4 (1A): now also J3.1 (Pin_1)
- net at A1.5 (2A): now also J3.4 (Pin_4)
- net at A1.6 (2B): now also J3.6 (Pin_6)
Changed lines of the file:
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@@
+	(wire
+		(pts
+			(xy 153.67 99.06) (xy 157.48 99.06)
+		)
+		(stroke
+			(width 0)
+			(type default)
+		)
+	)
 	(wire
 		(pts
@@
 	(wire
 		(pts
+			(xy 160.02 106.68) (xy 160.02 96.52)
+		)
+		(stroke
+			(width 0)
+			(type default)
+		)
+	)
+	(wire
+		(pts
 			(xy 130.81 93.98) (xy 109.22 93.98)
 		)
@@
 	(wire
 		(pts
+			(xy 162.56 93.98) (xy 162.56 111.76)
+		)
+		(stroke
+			(width 0)
+			(type default)
+		)
+	)
+	(wire
+		(pts
 			(xy 97.79 109.22) (xy 114.3 109.22)
 		)
@@
 	(wire
 		(pts
-			(xy 168.91 99.06) (xy 153.67 99.06)
-		)
-		(stroke
-			(width 0)
-			(type default)
-		)
-	)
-	(wire
-		(pts
 			(xy 102.87 76.2) (xy 102.87 88.9)
 		)
@@
 	(wire
 		(pts
-			(xy 168.91 93.98) (xy 153.67 93.98)
-		)
-		(stroke
-			(width 0)
-			(type default)
-		)
-	)
-	(wire
-		(pts
-			(xy 168.91 101.6) (xy 153.67 101.6)
-		)
-		(stroke
-			(width 0)
-			(type default)
-		)
-	)
-	(wire
-		(pts
-			(xy 168.91 96.52) (xy 153.67 96.52)
+			(xy 160.02 96.52) (xy 153.67 96.52)
+		)
+		(stroke
+			(width 0)
+			(type default)
+		)
+	)
+	(wire
+		(pts
+			(xy 153.67 93.98) (xy 162.56 93.98)
+		)
+		(stroke
+			(width 0)
+			(type default)
+		)
+	)
+	(wire
+		(pts
+			(xy 153.67 119.38) (xy 170.18 119.38)
 		)
 		(stroke
@@
 	(wire
 		(pts
+			(xy 170.18 106.68) (xy 160.02 106.68)
+		)
+		(stroke
+			(width 0)
+			(type default)
+		)
+	)
+	(wire
+		(pts
+			(xy 157.48 114.3) (xy 170.18 114.3)
+		)
+		(stroke
+			(width 0)
+			(type default)
+		)
+	)
+	(wire
+		(pts
 			(xy 120.65 64.77) (xy 120.65 68.58)
 		)
@@
 	(wire
 		(pts
+			(xy 162.56 111.76) (xy 170.18 111.76)
+		)
+		(stroke
+			(width 0)
+			(type default)
+		)
+	)
+	(wire
+		(pts
 			(xy 114.3 124.46) (xy 140.97 124.46)
 		)
@@
 	(wire
 		(pts
+			(xy 153.67 101.6) (xy 153.67 119.38)
+		)
+		(stroke
+			(width 0)
+			(type default)
+		)
+	)
+	(wire
+		(pts
 			(xy 140.97 72.39) (xy 140.97 78.74)
 		)
@@
 			(type default)
 			(color 48 16 255 1)
+		)
+	)
+	(wire
+		(pts
+			(xy 157.48 99.06) (xy 157.48 114.3)
+		)
+		(stroke
+			(width 0)
+			(type default)
 		)
 	)
@@
 	)
 	(symbol
+		(lib_id "Connector:Conn_01x06_Socket")
+		(at 175.26 111.76 0)
+		(unit 1)
+		(exclude_from_sim no)
+		(in_bom yes)
+		(on_board yes)
+		(dnp no)
+		(fields_autoplaced yes)
+		(property "Reference" "J3"
+			(at 176.53 111.7599 0)
+			(effects
+				(font
+					(size 1.27 1.27)
+				)
+				(justify left)
+			)
+		)
+		(property "Value" "Connecteur moteur  pas a pas"
+			(at 176.53 114.2999 0)
+			(effects
+				(font
+					(size 1.27 1.27)
+				)
+				(justify left)
+			)
+		)
+		(property "Footprint" "Connector_JST:JST_PH_B6B-PH-K_1x06_P2.00mm_Vertical"
+			(at 175.26 111.76 0)
+			(effects
+				(font
+					(size 1.27 1.27)
+				)
+				(hide yes)
+			)
+		)
+		(property "Datasheet" "~"
+			(at 175.26 111.76 0)
+			(effects
+				(font
+					(size 1.27 1.27)
+				)
+				(hide yes)
+			)
+		)
+		(property "Description" "Generic connector, single row, 01x06, script generated"
+			(at 175.26 111.76 0)
+			(effects
+				(font
+					(size 1.27 1.27)
+				)
+				(hide yes)
+			)
+		)
+		(pin "5"
+		)
+		(pin "1"
+		)
+		(pin "4"
+		)
+		(pin "3"
+		)
+		(pin "2"
+		)
+		(pin "6"
+		)
+		(instances
+			(project ""
+				(path "/55415806-8c1c-48ca-92ef-7c441d9b7337/8cf5d13e-b432-4713-b6ed-77f159fa5667"
+					(reference "J3")
+					(unit 1)
+				)
+			)
+		)
+	)
+	(symbol
 		(lib_id "Device:R")
 		(at 114.3 116.84 0)
@@
 					(unit 1)
 				)
-			)
-		)
-	)
-	(symbol
-		(lib_id "Connector:Conn_01x04_Socket")
-		(at 173.99 96.52 0)
-		(unit 1)
-		(exclude_from_sim no)
-		(in_bom yes)
-		(on_board yes)
-		(dnp no)
-		(property "Reference" "J1"
-			(at 176.276 97.79 0)
-			(effects
-				(font
-					(size 1.27 1.27)
-				)
-			)
-		)
-		(property "Value" "Connecteur moteur  pas a pas"
-			(at 170.942 104.14 0)
-			(effects
-				(font
-					(size 1.27 1.27)
-				)
-			)
-		)
-		(property "Footprint" "Connector_JST:JST_PH_B6B-PH-K_1x06_P2.00mm_Vertical"
-			(at 173.99 96.52 0)
-			(effects
-				(font
-					(size 1.27 1.27)
-				)
-				(hide yes)
-			)
-		)
-		(property "Datasheet" "~"
-			(at 173.99 96.52 0)
-			(effects
-				(font
-					(size 1.27 1.27)
-				)
-				(hide yes)
-			)
-		)
-		(property "Description" "Generic connector, single row, 01x04, script generated"
-			(at 173.99 96.52 0)
-			(effects
-				(font
-					(size 1.27 1.27)
-				)
-				(hide yes)
-			)
-		)
-		(pin "4"
-		)
-		(pin "2"
-		)
-		(pin "3"
-		)
-		(pin "1"
-		)
-		(instances
-			(project "medbox"
-				(path "/55415806-8c1c-48ca-92ef-7c441d9b7337/8cf5d13e-b432-4713-b6ed-77f159fa5667"
-					(reference "J1")
-					(unit 1)
-				)

Commit message: PCB me parrait OK
Parts:
- C1: footprint Capacitor_THT:CP_Radial_D6.3mm_P2.50mm -> Capacitor_THT:CP_Radial_D10.0mm_P5.00mm
- C2, C3: footprint Capacitor_THT:C_Disc_D5.0mm_W2.5mm_P2.50mm -> Capacitor_THT:C_Disc_D6.0mm_W2.5mm_P5.00mm
Connections:
- net +12V: now also C1.1; no longer C1.2
- net +3V3: now also R3.2, R9.2; no longer R3.1, R9.1
- net GND: now also C1.2, R13.1; no longer C1.1, R13.2
- net MOT_ENABLED: now also R3.1; no longer R3.2
- net MOT_MS1: now also R13.2; no longer R13.1
- net at J3.1 (Pin_1): now also A1.6 (2B); no longer A1.4 (1A)
- net at J3.3 (Pin_3): now also A1.5 (2A); no longer A1.3 (1B)
- net at J3.4 (Pin_4): now also A1.3 (1B); no longer A1.5 (2A)
- net at J3.6 (Pin_6): now also A1.4 (1A); no longer A1.6 (2B)
- net at A1.14 (~{SLEEP}): now also R9.1; no longer R9.2
Other:
- moved on the sheet: C1, R13, R3, R9
Changed lines of the file:
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@@
+	(wire
+		(pts
+			(xy 160.02 119.38) (xy 170.18 119.38)
+		)
+		(stroke
+			(width 0)
+			(type default)
+		)
+	)
 	(wire
 		(pts
@@
 	(wire
 		(pts
+			(xy 157.48 99.06) (xy 157.48 111.76)
+		)
+		(stroke
+			(width 0)
+			(type default)
+		)
+	)
+	(wire
+		(pts
 			(xy 114.3 109.22) (xy 114.3 113.03)
 		)
@@
 	(wire
 		(pts
+			(xy 162.56 93.98) (xy 162.56 114.3)
+		)
+		(stroke
+			(width 0)
+			(type default)
+		)
+	)
+	(wire
+		(pts
+			(xy 153.67 106.68) (xy 170.18 106.68)
+		)
+		(stroke
+			(width 0)
+			(type default)
+		)
+	)
+	(wire
+		(pts
 			(xy 130.81 86.36) (xy 120.65 86.36)
 		)
@@
 	(wire
 		(pts
-			(xy 160.02 106.68) (xy 160.02 96.52)
-		)
-		(stroke
-			(width 0)
-			(type default)
-		)
-	)
-	(wire
-		(pts
 			(xy 130.81 93.98) (xy 109.22 93.98)
 		)
@@
 	(wire
 		(pts
-			(xy 162.56 93.98) (xy 162.56 111.76)
-		)
-		(stroke
-			(width 0)
-			(type default)
-		)
-	)
-	(wire
-		(pts
 			(xy 97.79 109.22) (xy 114.3 109.22)
 		)
@@
 	(wire
 		(pts
+			(xy 153.67 101.6) (xy 153.67 106.68)
+		)
+		(stroke
+			(width 0)
+			(type default)
+		)
+	)
+	(wire
+		(pts
 			(xy 153.67 93.98) (xy 162.56 93.98)
 		)
@@
 	(wire
 		(pts
-			(xy 153.67 119.38) (xy 170.18 119.38)
+			(xy 160.02 96.52) (xy 160.02 119.38)
 		)
 		(stroke
@@
 	(wire
 		(pts
-			(xy 170.18 106.68) (xy 160.02 106.68)
-		)
-		(stroke
-			(width 0)
-			(type default)
-		)
-	)
-	(wire
-		(pts
-			(xy 157.48 114.3) (xy 170.18 114.3)
-		)
-		(stroke
-			(width 0)
-			(type default)
-		)
-	)
-	(wire
-		(pts
 			(xy 120.65 64.77) (xy 120.65 68.58)
 		)
@@
 	(wire
 		(pts
-			(xy 162.56 111.76) (xy 170.18 111.76)
-		)
-		(stroke
-			(width 0)
-			(type default)
-		)
-	)
-	(wire
-		(pts
 			(xy 114.3 124.46) (xy 140.97 124.46)
 		)
@@
 	(wire
 		(pts
-			(xy 153.67 101.6) (xy 153.67 119.38)
-		)
-		(stroke
-			(width 0)
-			(type default)
-		)
-	)
-	(wire
-		(pts
 			(xy 140.97 72.39) (xy 140.97 78.74)
 		)
@@
 	(wire
 		(pts
-			(xy 157.48 99.06) (xy 157.48 114.3)
-		)
-		(stroke
-			(width 0)
-			(type default)
-		)
-	)
-	(wire
-		(pts
 			(xy 163.83 86.36) (xy 177.8 86.36)
 		)
@@
 	(wire
 		(pts
+			(xy 157.48 111.76) (xy 170.18 111.76)
+		)
+		(stroke
+			(width 0)
+			(type default)
+		)
+	)
+	(wire
+		(pts
 			(xy 109.22 64.77) (xy 109.22 68.58)
 		)
@@
 			(type default)
 			(color 48 16 255 1)
+		)
+	)
+	(wire
+		(pts
+			(xy 162.56 114.3) (xy 170.18 114.3)
+		)
+		(stroke
+			(width 0)
+			(type default)
 		)
 	)
@@
 			)
 		)
-		(property "Footprint" "Capacitor_THT:C_Disc_D5.0mm_W2.5mm_P2.50mm"
+		(property "Footprint" "Capacitor_THT:C_Disc_D6.0mm_W2.5mm_P5.00mm"
 			(at 153.3652 80.01 0)
 			(effects
@@
 			)
 		)
-		(property "Footprint" "Capacitor_THT:C_Disc_D5.0mm_W2.5mm_P2.50mm"
+		(property "Footprint" "Capacitor_THT:C_Disc_D6.0mm_W2.5mm_P5.00mm"
 			(at 176.8348 68.58 0)
 			(effects
@@
 		)
 		(instances
-			(project ""
+			(project "medbox"
 				(path "/55415806-8c1c-48ca-92ef-7c441d9b7337/8cf5d13e-b432-4713-b6ed-77f159fa5667"
 					(reference "J3")
@@
 	(symbol
 		(lib_id "Device:R")
-		(at 109.22 72.39 0)
+		(at 109.22 72.39 180)
 		(unit 1)
 		(exclude_from_sim no)
@@
 		)
 		(property "Value" "R10K"
-			(at 111.506 72.644 90)
+			(at 106.934 72.136 90)
 			(effects
 				(font
@@
 		)
 		(property "Footprint" "Resistor_THT:R_Axial_DIN0207_L6.3mm_D2.5mm_P7.62mm_Horizontal"
-			(at 107.442 72.39 90)
+			(at 110.998 72.39 90)
 			(effects
 				(font
@@
 	(symbol
 		(lib_id "Device:C_Polarized")
-		(at 163.83 72.39 180)
+		(at 163.83 72.39 0)
+		(mirror y)
 		(unit 1)
 		(exclude_from_sim no)
@@
 		)
 		(property "Value" "C_Polarized 220µ"
-			(at 167.386 81.788 90)
+			(at 167.386 62.992 90)
 			(effects
 				(font
@@
 			)
 		)
-		(property "Footprint" "Capacitor_THT:CP_Radial_D6.3mm_P2.50mm"
-			(at 162.8648 68.58 0)
+		(property "Footprint" "Capacitor_THT:CP_Radial_D10.0mm_P5.00mm"
+			(at 162.8648 76.2 0)
 			(effects
 				(font
@@
 	(symbol
 		(lib_id "Device:R")
-		(at 102.87 72.39 0)
+		(at 102.87 72.39 180)
 		(unit 1)
 		(exclude_from_sim no)
@@
 		)
 		(property "Value" "R10K"
-			(at 105.664 72.39 90)
+			(at 100.076 72.39 90)
 			(effects
 				(font
@@
 		)
 		(property "Footprint" "Resistor_THT:R_Axial_DIN0207_L6.3mm_D2.5mm_P7.62mm_Horizontal"
-			(at 101.092 72.39 90)
+			(at 104.648 72.39 90)
 			(effects
 				(font
@@
 	(symbol
 		(lib_id "Device:R")
-		(at 104.14 116.84 0)
+		(at 104.14 116.84 180)
 		(unit 1)
 		(exclude_from_sim no)
@@
 		)
 		(property "Value" "R10K"
-			(at 101.346 116.84 90)
+			(at 106.934 116.84 90)
 			(effects
 				(font
@@
 		)
 		(property "Footprint" "Resistor_THT:R_Axial_DIN0207_L6.3mm_D2.5mm_P7.62mm_Horizontal"
-			(at 102.362 116.84 90)
-			(effects
-				(font
+			(at 105.918 116.84 90)
+			(effects
+				(font
